File: 1u_mixer.sch (EAGLE design)
At the start: 60 parts, among them IC1 TL072D, IC2 TL072D, IC3 TL072D, IC4 TL072D

Commit message: asd
Parts:
- C11, C12: device rcl:C-EUC0805 -> resistor:CPOL-EUE2-4
- C3, C4: device resistor:CPOL-EUE2-4 -> rcl:C-EUC0805
- renumbered +12V to +12, -12V to -12, IN1 to 1, IN2 to 2, IN3 to 3, IN4 to 4, IN5 to 5, IN6 to 6, LINE_OUT to LINE, MAIN_OUT to EURO, MASTER to VOL
Connections:
- net +12V: now also C1.+, C3.1; no longer C11.1, C9.+
- net -12V: now also C2.-, C4.2; no longer C10.-, C12.2
- net CH1: now also IC4B.OUT, R20.1, R21.2; no longer IC1B.OUT, R10.2, R13.1
- net CH2: now also IC4A.OUT, R17.1, R19.2; no longer IC1A.OUT, R12.2, R15.1
- net CH3: now also IC3B.OUT, R14.1, R15.2; no longer IC2B.OUT, R16.1, R6.2
- net CH4: now also IC3A.OUT, R11.1, R13.2; no longer IC2A.OUT, R17.1, R8.2
- net CH5: now also IC2B.OUT, R8.1, R9.2; no longer IC3B.OUT, R18.1, R2.2
- net CH6: now also IC2A.OUT, R5.1, R7.2; no longer IC3A.OUT, R19.1, R4.2
- net GND: now also C1.-, C2.+, C3.2, C4.1, IC4A.+IN, R4.1; no longer C10.+, C11.2, C12.1, C9.-, IC1A.+IN, R21.1
- net N$1: now also C7.+; no longer C1.+
- net N$10: now also C9.-; no longer C4.-
- net N$11: now also IC3B.-IN, R15.1, R16.2; no longer IC2B.-IN, R5.2, R6.1
- net N$12: now also R16.1; no longer R5.1
- net N$13: now also C10.+; no longer C5.+
- net N$14: now also C10.-; no longer C5.-
- net N$15: now also IC3A.-IN, R12.2, R13.1; no longer IC2A.-IN, R7.2, R8.1
- net N$16: now also R12.1; no longer R7.1
- net N$17: now also C11.+; no longer C6.+
- net N$18: now also C11.-; no longer C6.-
- net N$19: now also IC4B.-IN, R21.1, R22.2; no longer IC1B.-IN, R10.1, R9.2
- net N$2: now also C7.-; no longer C1.-
- net N$20: now also R22.1; no longer R9.1
- net N$21: now also C12.+; no longer C7.+
- net N$22: now also C12.-; no longer C7.-
- net N$23: now also IC4A.-IN, R18.2, R19.1; no longer IC1A.-IN, R11.2, R12.1
- net N$24: now also R18.1; no longer R11.1
- net N$25: now also R11.2, R14.2, R20.2, R5.2, R8.2; no longer R13.2, R15.2, R16.2, R18.2, R19.2
- net N$26: now also C5.-; no longer C2.-
- net N$27: now also C6.-; no longer C8.-
- net N$28: now also R2.1; no longer R14.1
- net N$29: now also IC1B.-IN, R1.1, R2.2; no longer IC4B.-IN, R14.2, R20.1
- net N$3: now also IC2B.-IN, R10.2, R9.1; no longer IC3B.-IN, R1.2, R2.1
- net N$30: now also C5.+, IC1B.OUT, R1.2, R3.1; no longer C2.+, IC4B.OUT, R20.2, R22.1
- net N$32: now also C6.+, IC1A.-IN, IC1A.OUT; no longer C8.+, IC4A.-IN, IC4A.OUT
- net N$33: now also IC1A.+IN, R3.2, R4.2; no longer IC4A.+IN, R21.2, R22.2
- net N$4: now also R10.1; no longer R1.1
- net N$5: now also C8.+; no longer C3.+
- net N$6: now also C8.-; no longer C3.-
- net N$7: now also IC2A.-IN, R6.2, R7.1; no longer IC3A.-IN, R3.2, R4.1
- net N$8: now also R6.1; no longer R3.1
- net N$9: now also C9.+; no longer C4.+
Other:
- moved on the sheet: C1, C10, C2, C5, C6, C7, C8, C9, IC1A, IC1B, IC2A, IC2B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

Commit message: 1vpcb
Parts:
- added C13, C14, C17, C18: (no value), resistor:CPOL-EUE2-4
- added C15, C16: (no value), rcl:C-EUC0805
- C11, C12, C7, C8: device resistor:CPOL-EUE2-4 -> rcl:C-EUC0805
Connections:
- net +12V: now also C12.1, C16.1, C8.1
- net -12V: now also C11.2, C15.2, C7.2
- net GND: now also C11.1, C12.2, C15.1, C16.2, C7.1, C8.2
- net N$1: now also C9.+; no longer C7.+
- net N$10: now also C13.-; no longer C9.-
- net N$13: now also C14.+; no longer C10.+
- net N$14: now also C14.-; no longer C10.-
- net N$17: now also C17.+; no longer C11.+
- net N$18: now also C17.-; no longer C11.-
- net N$2: now also C9.-; no longer C7.-
- net N$21: now also C18.+; no longer C12.+
- net N$22: now also C18.-; no longer C12.-
- net N$5: now also C10.+; no longer C8.+
- net N$6: now also C10.-; no longer C8.-
- net N$9: now also C13.+; no longer C9.+
Other:
- moved on the sheet: C10, C9

Commit message: values
Parts:
- R1: value (none) -> 100k
- R10, R12, R16, R18, R22, R6: value (none) -> 4k7
- R13, R15, R19, R2, R21, R4, R7, R9: value (none) -> 10k
- R3: value (none) -> 47k
Changed lines of the file:
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@@
 <setting verticaltext="up"/>
 </settings>
-<grid distance="0.01" unitdist="inch" unit="inch" style="lines" multiple="1" display="no" altdistance="0.01" altunitdist="inch" altunit="inch"/>
+<grid distance="0.1" unitdist="inch" unit="inch" style="lines" multiple="1" display="no" altdistance="0.01" altunitdist="inch" altunit="inch"/>
 <layers>
 <layer number="1" name="Top" color="4" fill="1" visible="no" active="no"/>
@@
 <part name="LVL6" library="jasons_stuff" deviceset="ALPS_POT_SMALL" device=""/>
 <part name="VOL" library="jasons_stuff" deviceset="ALPS_POT_SMALL" device=""/>
-<part name="R10" library="rcl" deviceset="R-EU_" device="R0805"/>
+<part name="R10" library="rcl" deviceset="R-EU_" device="R0805" value="4k7"/>
 <part name="GND2" library="supply1" deviceset="GND" device=""/>
-<part name="R9" library="rcl" deviceset="R-EU_" device="R0805"/>
+<part name="R9" library="rcl" deviceset="R-EU_" device="R0805" value="10k"/>
 <part name="C10" library="resistor" deviceset="CPOL-EU" device="E2-4"/>
-<part name="R6" library="rcl" deviceset="R-EU_" device="R0805"/>
+<part name="R6" library="rcl" deviceset="R-EU_" device="R0805" value="4k7"/>
 <part name="GND1" library="supply1" deviceset="GND" device=""/>
-<part name="R7" library="rcl" deviceset="R-EU_" device="R0805"/>
+<part name="R7" library="rcl" deviceset="R-EU_" device="R0805" value="10k"/>
 <part name="C13" library="resistor" deviceset="CPOL-EU" device="E2-4"/>
-<part name="R16" library="rcl" deviceset="R-EU_" device="R0805"/>
+<part name="R16" library="rcl" deviceset="R-EU_" device="R0805" value="4k7"/>
 <part name="GND3" library="supply1" deviceset="GND" device=""/>
-<part name="R15" library="rcl" deviceset="R-EU_" device="R0805"/>
+<part name="R15" library="rcl" deviceset="R-EU_" device="R0805" value="10k"/>
 <part name="C14" library="resistor" deviceset="CPOL-EU" device="E2-4"/>
-<part name="R12" library="rcl" deviceset="R-EU_" device="R0805"/>
+<part name="R12" library="rcl" deviceset="R-EU_" device="R0805" value="4k7"/>
 <part name="GND4" library="supply1" deviceset="GND" device=""/>
-<part name="R13" library="rcl" deviceset="R-EU_" device="R0805"/>
+<part name="R13" library="rcl" deviceset="R-EU_" device="R0805" value="10k"/>
 <part name="C17" library="resistor" deviceset="CPOL-EU" device="E2-4"/>
-<part name="R22" library="rcl" deviceset="R-EU_" device="R0805"/>
+<part name="R22" library="rcl" deviceset="R-EU_" device="R0805" value="4k7"/>
 <part name="GND5" library="supply1" deviceset="GND" device=""/>
-<part name="R21" library="rcl" deviceset="R-EU_" device="R0805"/>
+<part name="R21" library="rcl" deviceset="R-EU_" device="R0805" value="10k"/>
 <part name="C18" library="resistor" deviceset="CPOL-EU" device="E2-4"/>
-<part name="R18" library="rcl" deviceset="R-EU_" device="R0805"/>
+<part name="R18" library="rcl" deviceset="R-EU_" device="R0805" value="4k7"/>
 <part name="GND6" library="supply1" deviceset="GND" device=""/>
-<part name="R19" library="rcl" deviceset="R-EU_" device="R0805"/>
+<part name="R19" library="rcl" deviceset="R-EU_" device="R0805" value="10k"/>
 <part name="IC3" library="linear" deviceset="TL072" device="D"/>
 <part name="IC2" library="linear" deviceset="TL072" device="D"/>
@@
 <part name="R5" library="rcl" deviceset="R-EU_" device="R0805"/>
 <part name="GND8" library="supply1" deviceset="GND" device=""/>
-<part name="R2" library="rcl" deviceset="R-EU_" device="R0805"/>
-<part name="R1" library="rcl" deviceset="R-EU_" device="R0805"/>
+<part name="R2" library="rcl" deviceset="R-EU_" device="R0805" value="10k"/>
+<part name="R1" library="rcl" deviceset="R-EU_" device="R0805" value="100k"/>
 <part name="C5" library="resistor" deviceset="CPOL-EU" device="E2-4"/>
 <part name="C6" library="resistor" deviceset="CPOL-EU" device="E2-4"/>
 <part name="GND7" library="supply1" deviceset="GND" device=""/>
-<part name="R4" library="rcl" deviceset="R-EU_" device="R0805"/>
-<part name="R3" library="rcl" deviceset="R-EU_" device="R0805"/>
+<part name="R4" library="rcl" deviceset="R-EU_" device="R0805" value="10k"/>
+<part name="R3" library="rcl" deviceset="R-EU_" device="R0805" value="47k"/>
 <part name="GND9" library="supply1" deviceset="GND" device=""/>
 <part name="GND10" library="supply1" deviceset="GND" device=""/>

Commit message: V1
Other:
- note added: "SIX4MIX 6:1 AUDIO MIXER VERSION 1.A (2021)"
Changed lines of the file:
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@@
 <text x="398.78" y="298.45" size="2.54" layer="97">Signal passes through a 1/5 voltage
 divider and unity buffered for line out</text>
+<text x="283.21" y="267.97" size="5.08" layer="97">SIX4MIX 6:1 AUDIO MIXER
+VERSION 1.A (2021)</text>
 </plain>
 <instances>
