File: hardware/six4mix.brd (EAGLE design)
At the start: 160.3 x 20 mm, 66 parts, among them IC1 TL072D, IC2 TL072D, IC3 TL072D, IC4 TL072D

Commit message: id inputs A-F
Parts:
- renumbered 1 to A, 2 to B, 3 to C, 4 to D, 5 to E, 6 to F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
