File: stencil/six4mix_stencil.brd (EAGLE design)
At the start: 180 x 120 mm, 396 parts, among them IC1 TL072D, IC10 TL072D, IC11 TL072D, IC12 TL072D, IC13 TL072D, IC14 TL072D, IC15 TL072D, IC16 TL072D, IC17 TL072D, IC18 TL072D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

Commit message: stencil
Other:
- board size 180 x 120 mm -> 190 x 130 mm
