File: six4mix_power/six4mix_power.brd (EAGLE design)
At the start: 25.7 x 16.2 mm, 4 parts

Commit message: Update six4mix_power.brd
Parts:
- moved U$1 2.54 mm to (14.0, 8.89), turned to 270 degrees
Routing:
- net N$2: track 33.4 -> 10.2 mm
- net N$1: track 16.3 -> 26.1 mm
Other:
- board size 25.7 x 16.2 mm -> 25.4 x 16.2 mm
Changed lines of the file:
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@@
 <board>
 <plain>
-<wire x1="1.8415" y1="0.635" x2="26.3525" y2="0.635" width="0.3048" layer="20"/>
-<wire x1="1.016" y1="16.256" x2="1.016" y2="1.2065" width="0.3048" layer="20"/>
-<wire x1="1.016" y1="1.2065" x2="1.8415" y2="0.635" width="0.3048" layer="20" curve="90"/>
-<wire x1="1.016" y1="16.256" x2="1.9685" y2="16.8275" width="0.3048" layer="20" curve="-90"/>
+<wire x1="1.7145" y1="0.635" x2="26.3525" y2="0.635" width="0.3048" layer="20"/>
+<wire x1="1.27" y1="16.256" x2="1.27" y2="1.2065" width="0.3048" layer="20"/>
+<wire x1="1.27" y1="1.2065" x2="1.7145" y2="0.635" width="0.3048" layer="20" curve="90"/>
+<wire x1="1.27" y1="16.256" x2="1.9685" y2="16.8275" width="0.3048" layer="20" curve="-90"/>
 <wire x1="1.9685" y1="16.8275" x2="26.2255" y2="16.8275" width="0.3048" layer="20"/>
 <wire x1="26.2255" y1="16.8275" x2="26.67" y2="16.256" width="0.3048" layer="20" curve="-90"/>
@@
 <wire x1="26.67" y1="16.256" x2="26.67" y2="0.9525" width="0.3048" layer="20"/>
 <wire x1="26.67" y1="0.9525" x2="26.3525" y2="0.635" width="0.3048" layer="20" curve="-90"/>
-<wire x1="5.207" y1="13.462" x2="6.223" y2="13.462" width="0.4064" layer="52"/>
-<wire x1="5.207" y1="10.795" x2="6.223" y2="10.795" width="0.4064" layer="52"/>
-<wire x1="5.715" y1="10.2235" x2="5.715" y2="11.303" width="0.4064" layer="52"/>
-<polygon width="0.6096" layer="22">
-<vertex x="7.62" y="13.335"/>
-<vertex x="7.62" y="4.445"/>
-<vertex x="8.89" y="4.445"/>
-<vertex x="8.89" y="13.335"/>
+<wire x1="5.207" y1="13.462" x2="6.223" y2="13.462" width="0.4064" layer="51"/>
+<wire x1="5.207" y1="10.795" x2="6.223" y2="10.795" width="0.4064" layer="51"/>
+<wire x1="5.715" y1="10.2235" x2="5.715" y2="11.303" width="0.4064" layer="51"/>
+<polygon width="0.6096" layer="21">
+<vertex x="22.479" y="13.335"/>
+<vertex x="22.479" y="4.445"/>
+<vertex x="21.209" y="4.445"/>
+<vertex x="21.209" y="13.335"/>
 </polygon>
-<text x="3.302" y="4.191" size="1.27" layer="21" font="vector" ratio="20">RED</text>
-<text x="6.35" y="7.112" size="1.27" layer="22" font="vector" ratio="20" rot="R90">GD</text>
-<text x="3.302" y="2.54" size="1.27" layer="21" font="vector" ratio="20">STRIPE</text>
-<text x="13.462" y="14.605" size="1.27" layer="21" font="vector" ratio="20">1U ADAPT V1</text>
-<text x="14.605" y="1.397" size="1.27" layer="21" font="vector" ratio="20">six4pix.com</text>
+<text x="24.511" y="4.191" size="1.27" layer="21" font="vector" ratio="20" rot="R90">RED</text>
+<text x="6.35" y="7.112" size="1.27" layer="51" font="vector" ratio="20" rot="R90">GD</text>
+<text x="26.035" y="4.191" size="1.27" layer="21" font="vector" ratio="20" rot="R90">STRIPE</text>
+<text x="25.781" y="14.859" size="1.27" layer="22" font="vector" ratio="20" rot="MR0">1U ADAPT V1</text>
+<text x="13.335" y="1.397" size="1.27" layer="22" font="vector" ratio="20" rot="MR0">six4pix.com</text>
 </plain>
 <attributes>
@@
 <attribute name="VALUE" x="4.445" y="10.16" size="1.27" layer="28" rot="MR0"/>
 </element>
-<element name="U$1" library="jason_eagle6" package="2X5SMT" value="2X5SMT" x="16.51" y="8.89" smashed="yes" rot="R90"/>
+<element name="U$1" library="jason_eagle6" package="2X5SMT" value="2X5SMT" x="13.97" y="8.89" smashed="yes" rot="R270"/>
 </elements>
 <signals>
@@
 <contactref element="U$1" pad="10"/>
 <contactref element="-12" pad="1"/>
-<wire x1="11.43" y1="10.16" x2="11.43" y2="11.43" width="0.8128" layer="1"/>
-<wire x1="11.43" y1="6.35" x2="11.43" y2="11.43" width="0.8128" layer="1"/>
-<wire x1="3.175" y1="13.335" x2="11.049" y2="13.335" width="0.8128" layer="1"/>
-<wire x1="11.049" y1="13.335" x2="11.43" y2="12.954" width="0.8128" layer="1"/>
-<wire x1="11.43" y1="12.954" x2="11.43" y2="11.43" width="0.8128" layer="1"/>
+<wire x1="3.175" y1="13.335" x2="3.175" y2="14.605" width="0.8128" layer="1"/>
+<wire x1="3.175" y1="14.605" x2="3.81" y2="15.24" width="0.8128" layer="1"/>
+<wire x1="3.81" y1="15.24" x2="18.669" y2="15.24" width="0.8128" layer="1"/>
+<wire x1="18.669" y1="15.24" x2="19.05" y2="14.859" width="0.8128" layer="1"/>
+<wire x1="19.05" y1="14.859" x2="19.05" y2="11.43" width="0.8128" layer="1"/>
+<wire x1="19.05" y1="11.43" x2="19.05" y2="6.35" width="0.8128" layer="1"/>
 </signal>
 <signal name="N$2">
@@
 <contactref element="U$1" pad="5"/>
 <contactref element="+12" pad="1"/>
-<wire x1="3.175" y1="10.795" x2="5.207" y2="10.795" width="0.8128" layer="1"/>
-<wire x1="5.207" y1="10.795" x2="5.461" y2="10.541" width="0.8128" layer="1"/>
-<wire x1="5.461" y1="10.541" x2="5.461" y2="3.683" width="0.8128" layer="1"/>
-<wire x1="5.461" y1="3.683" x2="5.842" y2="3.302" width="0.8128" layer="1"/>
-<wire x1="5.842" y1="3.302" x2="21.209" y2="3.302" width="0.8128" layer="1"/>
-<wire x1="21.209" y1="3.302" x2="21.59" y2="3.683" width="0.8128" layer="1"/>
-<wire x1="21.59" y1="3.683" x2="21.59" y2="6.35" width="0.8128" layer="1"/>
-<wire x1="21.59" y1="11.43" x2="21.59" y2="6.35" width="0.8128" layer="1"/>
+<wire x1="3.175" y1="10.795" x2="8.89" y2="10.795" width="0.8128" layer="1"/>
+<wire x1="8.89" y1="6.35" x2="8.89" y2="10.795" width="0.8128" layer="1"/>
+<wire x1="8.89" y1="10.795" x2="8.89" y2="11.43" width="0" layer="19" extent="1-1"/>
 </signal>
 <signal name="GND">
@@
 <contactref element="GND" pad="1"/>
 <polygon width="0.3048" layer="1">
-<vertex x="1.016" y="16.891"/>
+<vertex x="1.524" y="16.764"/>
 <vertex x="26.67" y="16.764"/>
 <vertex x="26.67" y="0.762"/>
-<vertex x="1.016" y="0.889"/>
+<vertex x="1.524" y="0.762"/>
 </polygon>
 </signal>
